Commit message: feat: improve Mecanum spawn lifecycle and contract plugin
Strengthen model lifecycle handling in spawn launch and the Mecanum
Gazebo contract plugin on the current noetic release train.

File: models/xgc2_mecanum_ugv/model.sdf.xacro (robot description, xacro)
@@ -3,4 +3,6 @@
   <xacro:arg name="robot_namespace" default="ugv1"/>
   <xacro:arg name="drive_model" default="high_fidelity"/>
+  <xacro:arg name="plugin_filename" default="libgazebo_sim_mecanum_contract.so"/>
+  <xacro:arg name="mesh_prefix" default="model://mecanum_description/meshes"/>
   <xacro:property name="xgc_pi" value="3.141592653589793"/>
   <xacro:property name="high_fidelity" value="${'$(arg drive_model)' == 'high_fidelity'}"/>
@@ -75,5 +77,5 @@
       <visual name="base_link">
         <pose>0 0 0.05 0 0 0</pose>
-        <geometry><mesh><uri>model://mecanum_description/meshes/nexus_base_link.STL</uri><scale>0.001 0.001 0.001</scale></mesh></geometry>
+        <geometry><mesh><uri>$(arg mesh_prefix)/nexus_base_link.STL</uri><scale>0.001 0.001 0.001</scale></mesh></geometry>
         <material><ambient>0.9 0.8 0.6 1</ambient><diffuse>0.9 0.8 0.6 1</diffuse></material>
       </visual>
@@ -85,18 +87,18 @@
         </visual>
       </xacro:macro>
-      <xacro:fixed_visual name="upper_left_wheel_shaft" pose="0.150 0.108 0.05 0 0 0" uri="model://mecanum_description/meshes/wheel_shaft.STL" color="0.15 0.15 0.15 1"/>
-      <xacro:fixed_visual name="lower_left_wheel_shaft" pose="-0.150 0.108 0.05 0 0 0" uri="model://mecanum_description/meshes/wheel_shaft.STL" color="0.15 0.15 0.15 1"/>
-      <xacro:fixed_visual name="upper_right_wheel_shaft" pose="0.150 -0.108 0.05 ${xgc_pi} 0 0" uri="model://mecanum_description/meshes/wheel_shaft.STL" color="0.15 0.15 0.15 1"/>
-      <xacro:fixed_visual name="lower_right_wheel_shaft" pose="-0.150 -0.108 0.05 ${xgc_pi} 0 0" uri="model://mecanum_description/meshes/wheel_shaft.STL" color="0.15 0.15 0.15 1"/>
+      <xacro:fixed_visual name="upper_left_wheel_shaft" pose="0.150 0.108 0.05 0 0 0" uri="$(arg mesh_prefix)/wheel_shaft.STL" color="0.15 0.15 0.15 1"/>
+      <xacro:fixed_visual name="lower_left_wheel_shaft" pose="-0.150 0.108 0.05 0 0 0" uri="$(arg mesh_prefix)/wheel_shaft.STL" color="0.15 0.15 0.15 1"/>
+      <xacro:fixed_visual name="upper_right_wheel_shaft" pose="0.150 -0.108 0.05 ${xgc_pi} 0 0" uri="$(arg mesh_prefix)/wheel_shaft.STL" color="0.15 0.15 0.15 1"/>
+      <xacro:fixed_visual name="lower_right_wheel_shaft" pose="-0.150 -0.108 0.05 ${xgc_pi} 0 0" uri="$(arg mesh_prefix)/wheel_shaft.STL" color="0.15 0.15 0.15 1"/>
       <xacro:unless value="${high_fidelity}">
-        <xacro:fixed_visual name="upper_left_wheel" pose="0.150 0.150 0.05 0 0 0" uri="model://mecanum_description/meshes/mecanum_wheel_left.STL" color="0.6 0.6 0.6 1"/>
-        <xacro:fixed_visual name="lower_left_wheel" pose="-0.150 0.150 0.05 0 0 0" uri="model://mecanum_description/meshes/mecanum_wheel_right.STL" color="0.6 0.6 0.6 1"/>
-        <xacro:fixed_visual name="upper_right_wheel" pose="0.150 -0.150 0.05 ${xgc_pi} 0 0" uri="model://mecanum_description/meshes/mecanum_wheel_right.STL" color="0.6 0.6 0.6 1"/>
-        <xacro:fixed_visual name="lower_right_wheel" pose="-0.150 -0.150 0.05 ${xgc_pi} 0 0" uri="model://mecanum_description/meshes/mecanum_wheel_left.STL" color="0.6 0.6 0.6 1"/>
+        <xacro:fixed_visual name="upper_left_wheel" pose="0.150 0.150 0.05 0 0 0" uri="$(arg mesh_prefix)/mecanum_wheel_left.STL" color="0.6 0.6 0.6 1"/>
+        <xacro:fixed_visual name="lower_left_wheel" pose="-0.150 0.150 0.05 0 0 0" uri="$(arg mesh_prefix)/mecanum_wheel_right.STL" color="0.6 0.6 0.6 1"/>
+        <xacro:fixed_visual name="upper_right_wheel" pose="0.150 -0.150 0.05 ${xgc_pi} 0 0" uri="$(arg mesh_prefix)/mecanum_wheel_right.STL" color="0.6 0.6 0.6 1"/>
+        <xacro:fixed_visual name="lower_right_wheel" pose="-0.150 -0.150 0.05 ${xgc_pi} 0 0" uri="$(arg mesh_prefix)/mecanum_wheel_left.STL" color="0.6 0.6 0.6 1"/>
       </xacro:unless>
-      <xacro:fixed_visual name="front_sensor" pose="0.205 0 0.06 ${xgc_pi / 2.0} 0 0" uri="model://mecanum_description/meshes/urm04.STL" color="0.15 0.15 0.15 1"/>
-      <xacro:fixed_visual name="left_sensor" pose="0 0.108 0.06 ${xgc_pi / 2.0} 0 ${xgc_pi / 2.0}" uri="model://mecanum_description/meshes/urm04.STL" color="0.15 0.15 0.15 1"/>
-      <xacro:fixed_visual name="right_sensor" pose="0 -0.108 0.06 ${xgc_pi / 2.0} 0 ${-xgc_pi / 2.0}" uri="model://mecanum_description/meshes/urm04.STL" color="0.15 0.15 0.15 1"/>
-      <xacro:fixed_visual name="rear_sensor" pose="-0.201 0 0.06 ${xgc_pi / 2.0} 0 ${xgc_pi}" uri="model://mecanum_description/meshes/urm04.STL" color="0.15 0.15 0.15 1"/>
+      <xacro:fixed_visual name="front_sensor" pose="0.205 0 0.06 ${xgc_pi / 2.0} 0 0" uri="$(arg mesh_prefix)/urm04.STL" color="0.15 0.15 0.15 1"/>
+      <xacro:fixed_visual name="left_sensor" pose="0 0.108 0.06 ${xgc_pi / 2.0} 0 ${xgc_pi / 2.0}" uri="$(arg mesh_prefix)/urm04.STL" color="0.15 0.15 0.15 1"/>
+      <xacro:fixed_visual name="right_sensor" pose="0 -0.108 0.06 ${xgc_pi / 2.0} 0 ${-xgc_pi / 2.0}" uri="$(arg mesh_prefix)/urm04.STL" color="0.15 0.15 0.15 1"/>
+      <xacro:fixed_visual name="rear_sensor" pose="-0.201 0 0.06 ${xgc_pi / 2.0} 0 ${xgc_pi}" uri="$(arg mesh_prefix)/urm04.STL" color="0.15 0.15 0.15 1"/>
       <visual name="stereo_camera">
         <pose>0.205 0 0.06 0 0 0</pose>
@@ -106,10 +108,10 @@
     </link>
     <xacro:if value="${high_fidelity}">
-      <xacro:wheel name="upper_left_wheel" x="0.150" y="0.150" axis_y="1" roll="0" mesh="model://mecanum_description/meshes/mecanum_wheel_left.STL"/>
-      <xacro:wheel name="upper_right_wheel" x="0.150" y="-0.150" axis_y="-1" roll="${xgc_pi}" mesh="model://mecanum_description/meshes/mecanum_wheel_right.STL"/>
-      <xacro:wheel name="lower_left_wheel" x="-0.150" y="0.150" axis_y="1" roll="0" mesh="model://mecanum_description/meshes/mecanum_wheel_right.STL"/>
-      <xacro:wheel name="lower_right_wheel" x="-0.150" y="-0.150" axis_y="-1" roll="${xgc_pi}" mesh="model://mecanum_description/meshes/mecanum_wheel_left.STL"/>
+      <xacro:wheel name="upper_left_wheel" x="0.150" y="0.150" axis_y="1" roll="0" mesh="$(arg mesh_prefix)/mecanum_wheel_left.STL"/>
+      <xacro:wheel name="upper_right_wheel" x="0.150" y="-0.150" axis_y="-1" roll="${xgc_pi}" mesh="$(arg mesh_prefix)/mecanum_wheel_right.STL"/>
+      <xacro:wheel name="lower_left_wheel" x="-0.150" y="0.150" axis_y="1" roll="0" mesh="$(arg mesh_prefix)/mecanum_wheel_right.STL"/>
+      <xacro:wheel name="lower_right_wheel" x="-0.150" y="-0.150" axis_y="-1" roll="${xgc_pi}" mesh="$(arg mesh_prefix)/mecanum_wheel_left.STL"/>
     </xacro:if>
-    <plugin name="mecanum_contract" filename="libgazebo_sim_mecanum_contract.so">
+    <plugin name="mecanum_contract" filename="$(arg plugin_filename)">
       <robotNamespace>$(arg robot_namespace)</robotNamespace>
       <driveModel>$(arg drive_model)</driveModel>

Commit message: Use accepted low-polygon visuals in both Mecanum simulation modes

File: models/xgc2_mecanum_ugv/model.sdf.xacro (robot description, xacro)
@@ -20,5 +20,5 @@
       <visual name="visual">
         <pose>0 0 0 ${roll} 0 0</pose>
-        <geometry><mesh><uri>${mesh}</uri><scale>0.001 0.001 0.001</scale></mesh></geometry>
+        <geometry><mesh><uri>${mesh}</uri><scale>1 1 1</scale></mesh></geometry>
         <material><ambient>0.6 0.6 0.6 1</ambient><diffuse>0.6 0.6 0.6 1</diffuse></material>
       </visual>
@@ -77,5 +77,5 @@
       <visual name="base_link">
         <pose>0 0 0.05 0 0 0</pose>
-        <geometry><mesh><uri>$(arg mesh_prefix)/nexus_base_link.STL</uri><scale>0.001 0.001 0.001</scale></mesh></geometry>
+        <geometry><mesh><uri>$(arg mesh_prefix)/lod10k/nexus_base_link.dae</uri><scale>1 1 1</scale></mesh></geometry>
         <material><ambient>0.9 0.8 0.6 1</ambient><diffuse>0.9 0.8 0.6 1</diffuse></material>
       </visual>
@@ -83,22 +83,22 @@
         <visual name="${name}">
           <pose>${pose}</pose>
-          <geometry><mesh><uri>${uri}</uri><scale>0.001 0.001 0.001</scale></mesh></geometry>
+          <geometry><mesh><uri>${uri}</uri><scale>1 1 1</scale></mesh></geometry>
           <material><ambient>${color}</ambient><diffuse>${color}</diffuse></material>
         </visual>
       </xacro:macro>
-      <xacro:fixed_visual name="upper_left_wheel_shaft" pose="0.150 0.108 0.05 0 0 0" uri="$(arg mesh_prefix)/wheel_shaft.STL" color="0.15 0.15 0.15 1"/>
-      <xacro:fixed_visual name="lower_left_wheel_shaft" pose="-0.150 0.108 0.05 0 0 0" uri="$(arg mesh_prefix)/wheel_shaft.STL" color="0.15 0.15 0.15 1"/>
-      <xacro:fixed_visual name="upper_right_wheel_shaft" pose="0.150 -0.108 0.05 ${xgc_pi} 0 0" uri="$(arg mesh_prefix)/wheel_shaft.STL" color="0.15 0.15 0.15 1"/>
-      <xacro:fixed_visual name="lower_right_wheel_shaft" pose="-0.150 -0.108 0.05 ${xgc_pi} 0 0" uri="$(arg mesh_prefix)/wheel_shaft.STL" color="0.15 0.15 0.15 1"/>
+      <xacro:fixed_visual name="upper_left_wheel_shaft" pose="0.150 0.108 0.05 0 0 0" uri="$(arg mesh_prefix)/lod10k/wheel_shaft.dae" color="0.15 0.15 0.15 1"/>
+      <xacro:fixed_visual name="lower_left_wheel_shaft" pose="-0.150 0.108 0.05 0 0 0" uri="$(arg mesh_prefix)/lod10k/wheel_shaft.dae" color="0.15 0.15 0.15 1"/>
+      <xacro:fixed_visual name="upper_right_wheel_shaft" pose="0.150 -0.108 0.05 ${xgc_pi} 0 0" uri="$(arg mesh_prefix)/lod10k/wheel_shaft.dae" color="0.15 0.15 0.15 1"/>
+      <xacro:fixed_visual name="lower_right_wheel_shaft" pose="-0.150 -0.108 0.05 ${xgc_pi} 0 0" uri="$(arg mesh_prefix)/lod10k/wheel_shaft.dae" color="0.15 0.15 0.15 1"/>
       <xacro:unless value="${high_fidelity}">
-        <xacro:fixed_visual name="upper_left_wheel" pose="0.150 0.150 0.05 0 0 0" uri="$(arg mesh_prefix)/mecanum_wheel_left.STL" color="0.6 0.6 0.6 1"/>
-        <xacro:fixed_visual name="lower_left_wheel" pose="-0.150 0.150 0.05 0 0 0" uri="$(arg mesh_prefix)/mecanum_wheel_right.STL" color="0.6 0.6 0.6 1"/>
-        <xacro:fixed_visual name="upper_right_wheel" pose="0.150 -0.150 0.05 ${xgc_pi} 0 0" uri="$(arg mesh_prefix)/mecanum_wheel_right.STL" color="0.6 0.6 0.6 1"/>
-        <xacro:fixed_visual name="lower_right_wheel" pose="-0.150 -0.150 0.05 ${xgc_pi} 0 0" uri="$(arg mesh_prefix)/mecanum_wheel_left.STL" color="0.6 0.6 0.6 1"/>
+        <xacro:fixed_visual name="upper_left_wheel" pose="0.150 0.150 0.05 0 0 0" uri="$(arg mesh_prefix)/lod10k/mecanum_wheel_left.dae" color="0.6 0.6 0.6 1"/>
+        <xacro:fixed_visual name="lower_left_wheel" pose="-0.150 0.150 0.05 0 0 0" uri="$(arg mesh_prefix)/lod10k/mecanum_wheel_right.dae" color="0.6 0.6 0.6 1"/>
+        <xacro:fixed_visual name="upper_right_wheel" pose="0.150 -0.150 0.05 ${xgc_pi} 0 0" uri="$(arg mesh_prefix)/lod10k/mecanum_wheel_right.dae" color="0.6 0.6 0.6 1"/>
+        <xacro:fixed_visual name="lower_right_wheel" pose="-0.150 -0.150 0.05 ${xgc_pi} 0 0" uri="$(arg mesh_prefix)/lod10k/mecanum_wheel_left.dae" color="0.6 0.6 0.6 1"/>
       </xacro:unless>
-      <xacro:fixed_visual name="front_sensor" pose="0.205 0 0.06 ${xgc_pi / 2.0} 0 0" uri="$(arg mesh_prefix)/urm04.STL" color="0.15 0.15 0.15 1"/>
-      <xacro:fixed_visual name="left_sensor" pose="0 0.108 0.06 ${xgc_pi / 2.0} 0 ${xgc_pi / 2.0}" uri="$(arg mesh_prefix)/urm04.STL" color="0.15 0.15 0.15 1"/>
-      <xacro:fixed_visual name="right_sensor" pose="0 -0.108 0.06 ${xgc_pi / 2.0} 0 ${-xgc_pi / 2.0}" uri="$(arg mesh_prefix)/urm04.STL" color="0.15 0.15 0.15 1"/>
-      <xacro:fixed_visual name="rear_sensor" pose="-0.201 0 0.06 ${xgc_pi / 2.0} 0 ${xgc_pi}" uri="$(arg mesh_prefix)/urm04.STL" color="0.15 0.15 0.15 1"/>
+      <xacro:fixed_visual name="front_sensor" pose="0.205 0 0.06 ${xgc_pi / 2.0} 0 0" uri="$(arg mesh_prefix)/lod10k/urm04.dae" color="0.15 0.15 0.15 1"/>
+      <xacro:fixed_visual name="left_sensor" pose="0 0.108 0.06 ${xgc_pi / 2.0} 0 ${xgc_pi / 2.0}" uri="$(arg mesh_prefix)/lod10k/urm04.dae" color="0.15 0.15 0.15 1"/>
+      <xacro:fixed_visual name="right_sensor" pose="0 -0.108 0.06 ${xgc_pi / 2.0} 0 ${-xgc_pi / 2.0}" uri="$(arg mesh_prefix)/lod10k/urm04.dae" color="0.15 0.15 0.15 1"/>
+      <xacro:fixed_visual name="rear_sensor" pose="-0.201 0 0.06 ${xgc_pi / 2.0} 0 ${xgc_pi}" uri="$(arg mesh_prefix)/lod10k/urm04.dae" color="0.15 0.15 0.15 1"/>
       <visual name="stereo_camera">
         <pose>0.205 0 0.06 0 0 0</pose>
@@ -108,8 +108,8 @@
     </link>
     <xacro:if value="${high_fidelity}">
-      <xacro:wheel name="upper_left_wheel" x="0.150" y="0.150" axis_y="1" roll="0" mesh="$(arg mesh_prefix)/mecanum_wheel_left.STL"/>
-      <xacro:wheel name="upper_right_wheel" x="0.150" y="-0.150" axis_y="-1" roll="${xgc_pi}" mesh="$(arg mesh_prefix)/mecanum_wheel_right.STL"/>
-      <xacro:wheel name="lower_left_wheel" x="-0.150" y="0.150" axis_y="1" roll="0" mesh="$(arg mesh_prefix)/mecanum_wheel_right.STL"/>
-      <xacro:wheel name="lower_right_wheel" x="-0.150" y="-0.150" axis_y="-1" roll="${xgc_pi}" mesh="$(arg mesh_prefix)/mecanum_wheel_left.STL"/>
+      <xacro:wheel name="upper_left_wheel" x="0.150" y="0.150" axis_y="1" roll="0" mesh="$(arg mesh_prefix)/lod10k/mecanum_wheel_left.dae"/>
+      <xacro:wheel name="upper_right_wheel" x="0.150" y="-0.150" axis_y="-1" roll="${xgc_pi}" mesh="$(arg mesh_prefix)/lod10k/mecanum_wheel_right.dae"/>
+      <xacro:wheel name="lower_left_wheel" x="-0.150" y="0.150" axis_y="1" roll="0" mesh="$(arg mesh_prefix)/lod10k/mecanum_wheel_right.dae"/>
+      <xacro:wheel name="lower_right_wheel" x="-0.150" y="-0.150" axis_y="-1" roll="${xgc_pi}" mesh="$(arg mesh_prefix)/lod10k/mecanum_wheel_left.dae"/>
     </xacro:if>
     <plugin name="mecanum_contract" filename="$(arg plugin_filename)">
